File: Pintry-X2/CM4.kicad_sch (KiCad schematic)
At the start: 0 parts

Commit message: Bunch of shit done, probably should commit
Parts:
- added C1, C14, C16, C17, C5: 10uF, PintryParts-Footprints:C_0402_1005Metric, symbol Device:C_Small
- added C10, C8: 865080443007, Capacitor_SMD:CP_Elec_6.3x5.4, symbol PintryParts-Symbols:865080443007
- added C11, C12, C13, C15, C2, C3, C4, C7, C9: 0.1uF, PintryParts-Footprints:C_0402_1005Metric, symbol Device:C_Small
- added C6: 22uF, PintryParts-Footprints:C_0805_2012Metric, symbol Device:C_Small
- added D1, D15, D16, D2: DF2S6.2FS,L3M, Diode_SMD:D_SOD-923, symbol PintryParts-Symbols:DF2S6.2FS,L3M
- added D10, D11, D12, D3, D4, D5, D6, D7: D3V3M1U259-7, Diode_SMD:D_SOD-923, symbol PintryParts-Symbols:D3V3M1U259-7
- added D13, D14: DF2S16FS,L3M, Diode_SMD:D_SOD-923, symbol PintryParts-Symbols:DF2S16FS,L3M
- added D8, D9: APA2107SECK, PintryParts-Footprints:APA2107SECK, symbol PintryParts-Symbols:APA2107SECK
- added FB1, FB2: MPZ1608S101ATAH0, PintryParts-Footprints:L_0603_1608Metric, symbol PintryParts-Symbols:MPZ1608S101ATAH0
- added J1: USB_B_Micro, Connector_USB:USB_Micro-B_Amphenol_10103594-0001LF_Horizontal, symbol Connector:USB_B_Micro
- added J2: USB_A, Connector_USB:USB_A_Wuerth_614004134726_Horizontal, symbol Connector:USB_A
- added J3: JD0-0001NL, PintryParts-Footprints:Pulse-JD0-0001NL-0-0-MFG, symbol PintryParts-Symbols:JD0-0001NL
- added J4: DM3D-SF, Connector_Card:microSD_HC_Hirose_DM3D-SF, symbol Connector:Micro_SD_Card_Det
- added J5: UART, Connector_PinHeader_2.54mm:PinHeader_1x03_P2.54mm_Vertical, symbol Connector_Generic:Conn_01x03
- added J6: Expansion, symbol Connector_Generic:Conn_02x05_Odd_Even
- added J7, J8: Fan, Connector_Molex:Molex_KK-254_AE-6410-04A_1x04_P2.54mm_Vertical, symbol Connector_Generic:Conn_01x04
- added Module1: ComputeModule4-CM4, CM4IO:Raspberry-Pi-4-Compute-Module, symbol PintryParts-Symbols:ComputeModule4-CM4
- added Q1, Q2: BSS138PW, Package_TO_SOT_SMD:SOT-323_SC-70, symbol PintryParts-Symbols:BSS138PW
- added R1, R2, R5, R7, R8: 4K7, PintryParts-Footprints:R_0402_1005Metric, symbol Device:R_US
- added R10, R9: 100K, PintryParts-Footprints:R_0402_1005Metric, symbol Device:R_US
- added R3, R4: 470R, PintryParts-Footprints:R_0402_1005Metric, symbol Device:R_US
- added R6, R?: 1K, PintryParts-Footprints:R_0402_1005Metric, symbol Device:R_US
- added SW1: SW_Push, Button_Switch_THT:SW_Tactile_SPST_Angled_PTS645Vx58-2LFS, symbol Switch:SW_Push
- added TP?: GLOBAL_EN, TestPoint:TestPoint_Pad_D2.5mm, symbol Connector:TestPoint
- added TP?: RUN_PG, TestPoint:TestPoint_Pad_D2.5mm, symbol Connector:TestPoint
- added TP?: FAN1, TestPoint:TestPoint_Pad_D2.5mm, symbol Connector:TestPoint
- added TP?: VUSB, TestPoint:TestPoint_Pad_D2.5mm, symbol Connector:TestPoint
- added TP?: FAN0, TestPoint:TestPoint_Pad_D2.5mm, symbol Connector:TestPoint
- added U1: FSUSB30MUX, Package_SO:MSOP-10_3x3mm_P0.5mm, symbol PintryParts-Symbols:FSUSB30MUX
- added U2: MIC2005-0.5LYM5, Package_TO_SOT_SMD:SOT-23-5, symbol PintryParts-Symbols:MIC2005-0.5LYM5
- added U3: SN74LVC1G17, Package_TO_SOT_SMD:SOT-23-5, symbol PintryParts-Symbols:SN74LVC1G17
- added U4: 74AHCT1G126, Package_TO_SOT_SMD:SOT-353_SC-70-5, symbol 74xGxx:74AHCT1G126
- added U5, U6, U? (x2): TPD4EUSB30, Package_SON:USON-10_2.5x1.0mm_P0.5mm, symbol PintryParts-Symbols:TPD4EUSB30
Connections:
- new net: C17.1, D14.1 (K), FB2.1, J8.2 (Pin_2)
- new net: J3.14, R3.2
- new net: R?.2, U3.4
- new net: C6.1, C7.1, D2.1 (K), J2.1 (VBUS), TP?.1, U2.5 (VOUT)
- new net: Q1.1 (G), R7.2, R9.1
- new net: C9.1, J3.1
- new net: J3.12, R4.2
- new net: D8.1 (K), R?.1
- new net: C16.1, D13.1 (K), FB1.1, J7.2 (Pin_2)
- new net: D16.1 (K), J8.4 (Pin_4), Q2.3 (D), TP?.1
- new net: D9.1 (K), R6.1
- new net: R5.2, SW1.2
- new net: Q2.1 (G), R10.1, R8.2
- new net: D15.1 (K), J7.4 (Pin_4), Q1.3 (D), TP?.1
- new net: C10.1, C8.1, Module1.77 (+5v_(Input)), Module1.79 (+5v_(Input)), Module1.81 (+5v_(Input)), Module1.83 (+5v_(Input)), Module1.85 (+5v_(Input)), Module1.87 (+5v_(Input))
- new net +12V: FB1.2, FB2.2
- new net +3V3: C1.1, C11.1, C14.1, C15.1, C2.1, C3.1, D10.1 (K), D8.2 (A), D9.2 (A), J3.11, J3.13, J4.4 (VDD), Module1.78 (GPIO_VREF(1.8v/3.3v_Input)), Module1.84 (+3.3v_(Output)), Module1.86 (+3.3v_(Output)), SW1.1, U1.10 (VCC), U3.5 (VCC)
- new net +5V: C13.1, C4.1, C5.1, U2.1 (VIN), U2.3 (EN), U4.5 (VCC)
- new net ACT_LED: Module1.21 (PI_nLED_Activity), R6.2
- new net ETH_0_N: J3.3, Module1.10 (Ethernet_Pair0_N), U?.2 (D1-), U?.9
- new net ETH_0_P: J3.2, Module1.12 (Ethernet_Pair0_P), U?.1 (D1+), U?.10
- new net ETH_1_N: J3.5, Module1.6 (Ethernet_Pair1_N), U?.4 (D2+), U?.7
- new net ETH_1_P: J3.4, Module1.4 (Ethernet_Pair1_P), U?.5 (D2-), U?.6
- new net ETH_2_N: J3.7, Module1.9 (Ethernet_Pair2_N), U?.2 (D1-), U?.9
- new net ETH_2_P: J3.6, Module1.11 (Ethernet_Pair2_P), U?.1 (D1+), U?.10
- new net ETH_3_N: J3.9, Module1.5 (Ethernet_Pair3_N), U?.5 (D2-), U?.6
- new net ETH_3_P: J3.8, Module1.3 (Ethernet_Pair3_P), U?.4 (D2+), U?.7
- new net ETH_LEDG: Module1.17 (Ethernet_nLED2(3.3v)), R4.1
- new net ETH_LEDY: Module1.15 (Ethernet_nLED3(3.3v)), R3.1
- new net FAN0_PWM: Module1.31 (GPIO12), R8.1
- new net FAN1_PWM: Module1.28 (GPIO13), R7.1
- new net GLOBAL_EN: Module1.99 (Global_EN), TP?.1, U4.4
- new net GND: C1.2, C10.2, C11.2, C12.2, C13.2, C14.2, C15.2, C16.2, C17.2, C2.2, C3.2, C4.2, C5.2, C6.2, C7.2, C8.2, C9.2, D1.2 (A), D10.2 (A), D11.2 (A), D12.2 (A), D13.2 (A), D14.2 (A), D15.2 (A), D16.2 (A), D2.2 (A), D3.2 (A), D4.2 (A), D5.2 (A), D6.2 (A), D7.2 (A), J1.5 (GND), J1.6 (Shield), J2.4 (GND), J2.5 (Shield), J3.10, J3.S, J4.11 (SHIELD), J4.6 (VSS), J5.3 (Pin_3), J7.1 (Pin_1), J8.1 (Pin_1), Module1.1 (GND), Module1.107 (GND), Module1.108 (GND), Module1.113 (GND), Module1.114 (GND), Module1.119 (GND), Module1.120 (GND), Module1.125 (GND), Module1.126 (GND), Module1.13 (GND), Module1.131 (GND), Module1.132 (GND), Module1.137 (GND), Module1.138 (GND), Module1.14 (GND), Module1.144 (GND), Module1.150 (GND), Module1.155 (GND), Module1.156 (GND), Module1.161 (GND), Module1.162 (GND), Module1.167 (GND), Module1.168 (GND), Module1.173 (GND), Module1.174 (GND), Module1.179 (GND), Module1.180 (GND), Module1.185 (GND), Module1.186 (GND), Module1.191 (GND), Module1.192 (GND), Module1.197 (GND), Module1.198 (GND), Module1.2 (GND), Module1.22 (GND), Module1.23 (GND), Module1.32 (GND), Module1.33 (GND), Module1.42 (GND), Module1.43 (GND), Module1.52 (GND), Module1.53 (GND), Module1.59 (GND), Module1.60 (GND), Module1.65 (GND), Module1.66 (GND), Module1.7 (GND), Module1.71 (GND), Module1.74 (GND), Module1.8 (GND), Module1.98 (GND), Q1.2 (S), Q2.2 (S), R10.2, R2.2, R9.2, U1.5 (GND), U1.9 (~OE), U2.2 (GND), U3.3 (GND), U4.3 (GND), U5.3 (GND), U5.8 (GND), U6.3 (GND), U6.8 (GND), U?.3 (GND), U?.3 (GND), U?.8 (GND), U?.8 (GND)
- new net PCIe_CLK_N: Module1.112 (PCIe_CLK_N)
- new net PCIe_CLK_P: Module1.110 (PCIe_CLK_P)
- new net PCIe_RX_N: Module1.118 (PCIe_RX_N)
- new net PCIe_RX_P: Module1.116 (PCIe_RX_P)
- new net PCIe_TX_N: Module1.124 (PCIe_TX_N)
- new net PCIe_TX_P: Module1.122 (PCIe_TX_P)
- new net PI_POWER_SW: C12.1, D7.1 (K), Module1.25 (GPIO21), R5.1, U4.1
- new net PWR_LED: Module1.95 (nPI_LED_PWR), U3.2
- new net RUN_PG: Module1.92 (RUN_PG), TP?.1, U4.2
- new net RXD0: D11.1 (K), J5.1 (Pin_1), Module1.51 (GPIO15)
- new net SCL1: U6.5 (D2-), U6.6
- new net SDA1: Module1.58 (GPIO2), U6.4 (D2+), U6.7
- new net SD_CLK: J4.5 (CLK), Module1.57 (SD_CLK), U5.4 (D2+), U5.7
- new net SD_CMD: J4.3 (CMD), Module1.62 (SD_CMD), U5.5 (D2-), U5.6
- new net SD_DAT0: J4.7 (DAT0), Module1.63 (SD_DAT0), U6.1 (D1+), U6.10
- new net SD_DAT1: J4.8 (DAT1), Module1.67 (SD_DAT1), U6.2 (D1-), U6.9
- new net SD_DAT2: J4.1 (DAT2), Module1.69 (SD_DAT2), U5.1 (D1+), U5.10
- new net SD_DAT3: J4.2 (DAT3/CD), Module1.61 (SD_DAT3), U5.2 (D1-), U5.9
- new net TXD0: D12.1 (K), J5.2 (Pin_2), Module1.55 (GPIO14)
- new net USB1_N: D6.1 (K), J2.2 (D-), U1.8 (HSD1-)
- new net USB1_P: D4.1 (K), J2.3 (D+), U1.2 (HSD1+)
- new net USB2_N: D5.1 (K), J1.2 (D-), U1.7 (HSD2-)
- new net USB2_P: D3.1 (K), J1.3 (D+), U1.3 (HSD2+)
- new net USB_N: Module1.103 (USB2_N), U1.6 (D-)
- new net USB_OTG: Module1.101 (USB_OTG_ID), R1.2, R2.1, U1.1 (Sel)
- new net USB_P: Module1.105 (USB2_P), U1.4 (D+)
- new net VBUS_MICRO: D1.1 (K), J1.1 (VBUS), R1.1
- new net ~PCIe_RST: Module1.109 (PCIe_nRST)
- new net ~RPIBOOT: Module1.93 (nRPIBOOT)
- no-connect marks 0 -> 103
Other:
- note added: "0 HSD1"
- note added: "1 HSD2"
- note added: "Internal 1.8k pull-ups"
- note added: "Sel Out"
- company: (none) -> www.cezarchirila.com
- title: (none) -> Pintry X2
