File: Pintry-X2/Pintry-X2.kicad_pcb (KiCad board)
At the start: 0 parts

Commit message: Finished Shematic. Starting PCB
Parts:
- added C1: 10uF, PintryParts-Footprints:C_0402_1005Metric, F.Cu at (187.9, -136.1)
- added C10: 865080443007, Capacitor_SMD:CP_Elec_6.3x5.4, F.Cu at (171.2, -125.3)
- added C11: 0.1uF, PintryParts-Footprints:C_0402_1005Metric, F.Cu at (180.8, -127.3)
- added C12: 0.1uF, PintryParts-Footprints:C_0402_1005Metric, F.Cu at (184.8, -131.8)
- added C13: 0.1uF, PintryParts-Footprints:C_0402_1005Metric, F.Cu at (177.9, -125.3)
- added C14: 10uF, PintryParts-Footprints:C_0402_1005Metric, F.Cu at (177.9, -123.4)
- added C15: 0.1uF, PintryParts-Footprints:C_0402_1005Metric, F.Cu at (141.2, -86.8)
- added C16: 10uF, PintryParts-Footprints:C_0402_1005Metric, F.Cu at (136.0, -82.3)
- added C17: 10uF, PintryParts-Footprints:C_0402_1005Metric, F.Cu at (193.6, -138.6)
- added C18: 15pF, PintryParts-Footprints:C_0402_1005Metric, F.Cu at (229.1, -107.4)
- added C19: 0.01uF, PintryParts-Footprints:C_0402_1005Metric, F.Cu at (220.5, -99.5)
- added C2: 0.1uF, PintryParts-Footprints:C_0402_1005Metric, F.Cu at (224.1, -70.7)
- added C20: 0.01uF, PintryParts-Footprints:C_0402_1005Metric, F.Cu at (223.4, -103.5)
- added C23: 0.1uF, PintryParts-Footprints:C_0402_1005Metric, F.Cu at (217.5, -95.2)
- added C24: 10uF, PintryParts-Footprints:C_0402_1005Metric, F.Cu at (242.0, -118.7)
- added C27: 0.1uF, PintryParts-Footprints:C_0402_1005Metric, F.Cu at (232.0, -109.5)
- added C28: 0.1uF, PintryParts-Footprints:C_0402_1005Metric, F.Cu at (219.8, -101.5)
- added C29: 10uF, PintryParts-Footprints:C_0402_1005Metric, F.Cu at (243.7, -126.9)
- added C3: 0.1uF, PintryParts-Footprints:C_0402_1005Metric, F.Cu at (187.9, -134.2)
- added C30: 0.1uF, PintryParts-Footprints:C_0402_1005Metric, F.Cu at (211.7, -94.7)
- added C31: 0.1uF, PintryParts-Footprints:C_0402_1005Metric, F.Cu at (249.4, -126.9)
- added C32: 0.1uF, PintryParts-Footprints:C_0402_1005Metric, F.Cu at (243.7, -124.9)
- added C33: 0.1uF, PintryParts-Footprints:C_0402_1005Metric, F.Cu at (211.7, -96.6)
- added C34: 0.1uF, PintryParts-Footprints:C_0402_1005Metric, F.Cu at (246.6, -124.9)
- added C35: 0.1uF, PintryParts-Footprints:C_0402_1005Metric, F.Cu at (223.4, -105.4)
- added C36: 0.1uF, PintryParts-Footprints:C_0402_1005Metric, F.Cu at (211.7, -92.7)
- added C37: 0.1uF, PintryParts-Footprints:C_0402_1005Metric, F.Cu at (243.7, -122.9)
- added C38: 0.1uF, PintryParts-Footprints:C_0402_1005Metric, F.Cu at (220.5, -97.6)
- added C39: 0.1uF, PintryParts-Footprints:C_0402_1005Metric, F.Cu at (214.6, -92.7)
- added C4: 0.1uF, PintryParts-Footprints:C_0402_1005Metric, F.Cu at (221.2, -68.7)
- added C40: 0.1uF, PintryParts-Footprints:C_0402_1005Metric, F.Cu at (217.6, -97.1)
- added C41: 0.1uF, PintryParts-Footprints:C_0402_1005Metric, F.Cu at (226.3, -107.4)
- added C42: 0.1uF, PintryParts-Footprints:C_0402_1005Metric, F.Cu at (226.3, -105.5)
- added C43: 0.1uF, PintryParts-Footprints:C_0402_1005Metric, F.Cu at (211.7, -90.7)
- added C44: 0.1uF, PintryParts-Footprints:C_0402_1005Metric, F.Cu at (219.5, -110.6)
- added C45: 0.01uF, PintryParts-Footprints:C_0402_1005Metric, F.Cu at (246.6, -126.9)
- added C46: 0.01uF, PintryParts-Footprints:C_0402_1005Metric, F.Cu at (214.6, -96.6)
- added C47: 0.01uF, PintryParts-Footprints:C_0402_1005Metric, F.Cu at (258.8, -132.6)
- added C48: 0.01uF, PintryParts-Footprints:C_0402_1005Metric, F.Cu at (214.6, -94.7)
- added C49: 865080443007, Capacitor_SMD:CP_Elec_6.3x5.4, F.Cu at (226.3, -123.8)
- added C5: 10uF, PintryParts-Footprints:C_0402_1005Metric, F.Cu at (224.0, -68.7)
- added C50: 865080443007, Capacitor_SMD:CP_Elec_6.3x5.4, F.Cu at (215.6, -123.8)
- added C51: 0.01uF, PintryParts-Footprints:C_0402_1005Metric, F.Cu at (229.1, -109.4)
- added C52: 0.01uF, PintryParts-Footprints:C_0402_1005Metric, F.Cu at (226.3, -103.5)
- added C53: 0.01uF, PintryParts-Footprints:C_0402_1005Metric, F.Cu at (222.6, -101.5)
- added C54: 0.01uF, PintryParts-Footprints:C_0402_1005Metric, F.Cu at (243.7, -120.9)
- added C55: 865080443007, Capacitor_SMD:CP_Elec_6.3x5.4, F.Cu at (236.9, -123.8)
- added C56: 865080443007, Capacitor_SMD:CP_Elec_6.3x5.4, F.Cu at (215.6, -115.6)
- added C57: 0.1uF, PintryParts-Footprints:C_0402_1005Metric, F.Cu at (138.0, -61.1)
- added C58: 22uF, PintryParts-Footprints:C_0805_2012Metric, F.Cu at (143.0, -69.6)
- added C59: TBD, PintryParts-Footprints:C_0402_1005Metric, F.Cu at (142.2, -65.1)
- added C6: 22uF, PintryParts-Footprints:C_0805_2012Metric, F.Cu at (227.1, -74.7)
- added C60: 0.1uF, PintryParts-Footprints:C_0402_1005Metric, F.Cu at (129.8, -54.1)
- added C61: 1uF, PintryParts-Footprints:C_0402_1005Metric, F.Cu at (146.6, -68.8)
- added C62: 22uF, PintryParts-Footprints:C_0805_2012Metric, F.Cu at (147.4, -73.2)
- added C63: 22uF, PintryParts-Footprints:C_0805_2012Metric, F.Cu at (134.3, -64.1)
- added C64: 22uF, PintryParts-Footprints:C_0805_2012Metric, F.Cu at (134.3, -61.1)
- added C65: 0.1uF, PintryParts-Footprints:C_0402_1005Metric, F.Cu at (125.2, -49.5)
- added C66: 865080443007, Capacitor_SMD:CP_Elec_6.3x5.4, F.Cu at (109.6, -54.6)
- added C67: 10uF, PintryParts-Footprints:C_0402_1005Metric, F.Cu at (183.7, -129.8)
- added C68: 10uF, PintryParts-Footprints:C_0402_1005Metric, F.Cu at (190.8, -136.1)
- added C7: 0.1uF, PintryParts-Footprints:C_0402_1005Metric, F.Cu at (230.8, -75.2)
- added C8: 865080443007, Capacitor_SMD:CP_Elec_6.3x5.4, F.Cu at (121.9, -83.7)
- added C9: 0.1uF, PintryParts-Footprints:C_0402_1005Metric, F.Cu at (197.3, -143.2)
- added D1: DF2S6.2FS,L3M, Diode_SMD:D_SOD-923, F.Cu at (240.8, -82.9)
- added D10: D3V3M1U259-7, Diode_SMD:D_SOD-923, F.Cu at (141.1, -84.9)
- added D11: D3V3M1U259-7, Diode_SMD:D_SOD-923, F.Cu at (175.5, -120.3)
- added D12: D3V3M1U259-7, Diode_SMD:D_SOD-923, F.Cu at (166.5, -111.3)
- added D13: DF2S16FS,L3M, Diode_SMD:D_SOD-923, F.Cu at (197.2, -141.2)
- added D14: DF2S16FS,L3M, Diode_SMD:D_SOD-923, F.Cu at (180.8, -125.4)
- added D15: DF2S6.2FS,L3M, Diode_SMD:D_SOD-923, F.Cu at (170.8, -115.2)
- added D16: DF2S6.2FS,L3M, Diode_SMD:D_SOD-923, F.Cu at (136.0, -80.3)
- added D17: APA2107SECK, PintryParts-Footprints:APA2107SECK, F.Cu at (211.6, -110.2)
- added D2: DF2S6.2FS,L3M, Diode_SMD:D_SOD-923, F.Cu at (226.9, -72.2)
- added D20: DF2S6.2FS,L3M, Diode_SMD:D_SOD-923, F.Cu at (249.4, -124.9)
- added D21: DF2S16FS,L3M, Diode_SMD:D_SOD-923, F.Cu at (234.8, -109.5)
- added D22: DF2S6.2FS,L3M, Diode_SMD:D_SOD-923, F.Cu at (246.5, -122.9)
- added D23: DF2S16FS,L3M, Diode_SMD:D_SOD-923, F.Cu at (252.2, -126.9)
- added D24: BZX384-B13, Diode_SMD:D_SOD-323, F.Cu at (126.2, -55.6)
- added D25: DF2S16FS,L3M, Diode_SMD:D_SOD-923, F.Cu at (130.7, -60.6)
- added D26: BZX384-B13, Diode_SMD:D_SOD-323, F.Cu at (121.6, -51.0)
- added D3: D3V3M1U259-7, Diode_SMD:D_SOD-923, F.Cu at (226.8, -68.3)
- added D4: D3V3M1U259-7, Diode_SMD:D_SOD-923, F.Cu at (237.9, -80.1)
- added D5: D3V3M1U259-7, Diode_SMD:D_SOD-923, F.Cu at (230.7, -73.2)
- added D6: D3V3M1U259-7, Diode_SMD:D_SOD-923, F.Cu at (226.9, -70.2)
- added D7: D3V3M1U259-7, Diode_SMD:D_SOD-923, F.Cu at (187.6, -132.2)
- added D8: APA2107SECK, PintryParts-Footprints:APA2107SECK, F.Cu at (147.0, -93.2)
- added D9: APA2107SECK, PintryParts-Footprints:APA2107SECK, F.Cu at (184.9, -142.8)
- added FB1: MPZ1608S101ATAH0, PintryParts-Footprints:L_0603_1608Metric, F.Cu at (178.5, -131.6)
- added FB2: MPZ1608S101ATAH0, PintryParts-Footprints:L_0603_1608Metric, F.Cu at (190.2, -138.4)
- added FB3: MPZ1608S101ATAH0, PintryParts-Footprints:L_0603_1608Metric, F.Cu at (228.2, -111.6)
- added FB4: MPZ1608S101ATAH0, PintryParts-Footprints:L_0603_1608Metric, F.Cu at (212.3, -100.9)
- added FB5: MPZ1608S101ATAH0, PintryParts-Footprints:L_0603_1608Metric, F.Cu at (212.3, -103.4)
- added FB6: MPZ1608S101ATAH0, PintryParts-Footprints:L_0603_1608Metric, F.Cu at (216.3, -103.4)
- added FID1: Fiducial Top, Fiducial:Fiducial_1mm_Mask2mm, F.Cu at (182.9, -82.2)
- added FID2: Fiducial Bottom, Fiducial:Fiducial_1mm_Mask2mm, B.Cu at (177.7, -72.6)
- added FID3: Fiducial Top, Fiducial:Fiducial_1mm_Mask2mm, F.Cu at (188.8, -83.0)
- added FID4: Fiducial Bottom, Fiducial:Fiducial_1mm_Mask2mm, B.Cu at (189.2, -73.2)
- added FID5: Fiducial Top, Fiducial:Fiducial_1mm_Mask2mm, F.Cu at (177.0, -82.7)
- added FID6: Fiducial Bottom, Fiducial:Fiducial_1mm_Mask2mm, B.Cu at (183.6, -73.1)
- added FL1: DLW5BTM101SQ2L, PintryParts-Footprints:DLW5BTM101SQ2L, F.Cu at (119.5, -66.1)
- added H1: M3 MountingHole, PintryParts-Footprints:MountingHole_3.2mm_M3, F.Cu at (166.0, 206.0)
- added H2: M3 MountingHole, PintryParts-Footprints:MountingHole_3.2mm_M3, F.Cu at (74.0, 206.0)
- added H3: M3 MountingHole, PintryParts-Footprints:MountingHole_3.2mm_M3, F.Cu at (166.0, 114.0)
- added H4: M3 MountingHole, PintryParts-Footprints:MountingHole_3.2mm_M3, F.Cu at (74.0, 114.0)
- added J1: USB_B_Micro, PintryParts-Footprints:USB_Micro-B_Amphenol_10103594-0001LF_Horizontal, F.Cu at (211.0, -47.9)
- added J10: 1735284-3, PintryParts-Footprints:TE_1735284-3, B.Cu at (153.6, 160.0)
- added J11: 54-00131, PintryParts-Footprints:54-00131, F.Cu at (186.4, -55.5)
- added J12: Alternate Power Connector, Connector_Wire:SolderWire-1sqmm_1x02_P5.4mm_D1.4mm_OD2.7mm, F.Cu at (118.6, -72.3)
- added J2: USB_A, PintryParts-Footprints:USB_A_Amphenol_ICC_73725-11A0BLF_Horizontal, F.Cu at (197.4, -56.0)
- added J3: JD0-0001NL, PintryParts-Footprints:Pulse-JD0-0001NL-0-0-MFG, F.Cu at (155.8, -132.1)
- added J4: DM3D-SF, Connector_Card:microSD_HC_Hirose_DM3D-SF, F.Cu at (153.1, -113.2)
- added J5: UART, Connector_PinHeader_2.54mm:PinHeader_1x03_P2.54mm_Vertical, F.Cu at (162.9, -118.4)
- added J6: Expansion, Connector_PinHeader_2.54mm:PinHeader_2x05_P2.54mm_Vertical, F.Cu at (168.2, -141.9)
- added J7: Fan, Connector_Molex:Molex_KK-254_AE-6410-04A_1x04_P2.54mm_Vertical, F.Cu at (106.6, -83.9)
- added J8: Fan, Connector_Molex:Molex_KK-254_AE-6410-04A_1x04_P2.54mm_Vertical, F.Cu at (148.0, -98.5)
- added J9: 1735284-3, PintryParts-Footprints:TE_1735284-3, B.Cu at (112.5, 160.0)
- added L1: NRS5030T4R7MMGJ, PintryParts-Footprints:L_Taiyo-Yuden_NR-50xx, F.Cu at (260.7, -140.9)
- added L2: PA4341.122NLT, PintryParts-Footprints:Pulse_PA4341, F.Cu at (131.4, -70.4)
- added Module1: ComputeModule4-CM4, PintryParts-Footprints:Raspberry-Pi-4-Compute-Module, F.Cu at (103.5, 188.0)
- added Q1: BSS138PW, Package_TO_SOT_SMD:SOT-323_SC-70, F.Cu at (162.8, -109.2)
- added Q2: BSS138PW, Package_TO_SOT_SMD:SOT-323_SC-70, F.Cu at (172.0, -119.4)
- added Q5: SIA483DJ, Package_TO_SOT_SMD:Vishay_PowerPAK_SC70-6L_Single, F.Cu at (138.4, -63.8)
- added Q6: BC857BW, Package_TO_SOT_SMD:SOT-323_SC-70, F.Cu at (143.0, -72.9)
- added Q7: SIA483DJ, Package_TO_SOT_SMD:Vishay_PowerPAK_SC70-6L_Single, F.Cu at (125.9, -52.3)
- added R1: 1K, PintryParts-Footprints:R_0402_1005Metric, F.Cu at (114.5, -79.0)
- added R10: 100K, PintryParts-Footprints:R_0402_1005Metric, F.Cu at (181.9, -131.8)
- added R11: 4K7, PintryParts-Footprints:R_0402_1005Metric, F.Cu at (219.2, -106.6)
- added R12: 12K1, PintryParts-Footprints:R_0402_1005Metric, F.Cu at (220.5, -104.6)
- added R13: 12K1, PintryParts-Footprints:R_0402_1005Metric, F.Cu at (222.1, -107.4)
- added R14: 4K7, PintryParts-Footprints:R_0402_1005Metric, F.Cu at (216.6, -110.5)
- added R15: 100K, PintryParts-Footprints:R_0402_1005Metric, F.Cu at (177.9, -127.3)
- added R17: 4K7, PintryParts-Footprints:R_0402_1005Metric, F.Cu at (215.8, -101.1)
- added R18: 4K7, PintryParts-Footprints:R_0402_1005Metric, F.Cu at (214.7, -98.6)
- added R2: 4K7, PintryParts-Footprints:R_0402_1005Metric, F.Cu at (221.2, -70.7)
- added R21: 4K7, PintryParts-Footprints:R_0402_1005Metric, F.Cu at (211.8, -98.6)
- added R22: 100K, PintryParts-Footprints:R_0402_1005Metric, F.Cu at (133.7, -58.6)
- added R23: 100k, PintryParts-Footprints:R_0402_1005Metric, F.Cu at (108.7, -49.5)
- added R24: 100k, PintryParts-Footprints:R_0402_1005Metric, F.Cu at (129.8, -56.0)
- added R25: 100k, PintryParts-Footprints:R_0402_1005Metric, F.Cu at (124.4, -68.9)
- added R26: 100k, PintryParts-Footprints:R_0402_1005Metric, F.Cu at (111.6, -49.5)
- added R27: 4K7, PintryParts-Footprints:R_0402_1005Metric, F.Cu at (146.7, -70.7)
- added R28: 4K7, PintryParts-Footprints:R_0402_1005Metric, F.Cu at (142.2, -67.1)
- added R29: 221K, PintryParts-Footprints:R_0402_1005Metric, F.Cu at (132.7, -56.6)
- added R3: 470R, PintryParts-Footprints:R_0402_1005Metric, F.Cu at (108.7, -79.0)
- added R30: 30K1, PintryParts-Footprints:R_0402_1005Metric, F.Cu at (130.8, -58.6)
- added R31: 100k, PintryParts-Footprints:R_0402_1005Metric, F.Cu at (105.8, -49.5)
- added R32: 4K7, PintryParts-Footprints:R_0402_1005Metric, F.Cu at (240.8, -84.8)
- added R33: 0R, PintryParts-Footprints:R_0402_1005Metric, F.Cu at (219.2, -108.6)
- added R34: 0R, PintryParts-Footprints:R_0402_1005Metric, F.Cu at (217.6, -99.1)
- added R4: 470R, PintryParts-Footprints:R_0402_1005Metric, F.Cu at (159.3, -101.5)
- added R5: 4K7, PintryParts-Footprints:R_0402_1005Metric, F.Cu at (174.5, -131.8)
- added R6: 1K, PintryParts-Footprints:R_0402_1005Metric, F.Cu at (177.9, -129.3)
- added R7: 4K7, PintryParts-Footprints:R_0402_1005Metric, F.Cu at (111.6, -79.0)
- added R8: 4K7, PintryParts-Footprints:R_0402_1005Metric, F.Cu at (105.8, -79.0)
- added R9: 100K, PintryParts-Footprints:R_0402_1005Metric, F.Cu at (180.8, -129.3)
- added SW1: SW_Push, Button_Switch_THT:SW_Tactile_SPST_Angled_PTS645Vx58-2LFS, F.Cu at (176.1, -137.8)
- added TP1: VIN, TestPoint:TestPoint_Pad_D1.0mm, F.Cu at (117.2, -55.8)
- added TP10: FAN0, TestPoint:TestPoint_Pad_D1.0mm, F.Cu at (190.7, -141.9)
- added TP11: +1V2, TestPoint:TestPoint_Pad_D1.0mm, F.Cu at (212.6, -106.9)
- added TP14: VUSB, TestPoint:TestPoint_Pad_D1.0mm, F.Cu at (234.3, -78.8)
- added TP15: GND, TestPoint:TestPoint_Pad_D1.0mm, F.Cu at (121.8, -54.8)
- added TP16: GND, TestPoint:TestPoint_Pad_D1.0mm, F.Cu at (138.5, -72.5)
- added TP17: GND, TestPoint:TestPoint_Pad_D1.0mm, F.Cu at (138.5, -67.9)
- added TP18: 3V3, TestPoint:TestPoint_Pad_D1.0mm, F.Cu at (129.5, -81.1)
- added TP2: VCC, TestPoint:TestPoint_Pad_D1.0mm, F.Cu at (125.3, -63.9)
- added TP3: VIN_RP, TestPoint:TestPoint_Pad_D1.0mm, F.Cu at (129.8, -63.9)
- added TP4: +5V, TestPoint:TestPoint_Pad_D1.0mm, F.Cu at (127.0, -59.3)
- added TP5: +12V, TestPoint:TestPoint_Pad_D1.0mm, F.Cu at (122.5, -59.3)
- added TP6: GND, TestPoint:TestPoint_Pad_D1.0mm, F.Cu at (117.2, -51.2)
- added TP7: RUN_PG, TestPoint:TestPoint_Pad_D1.0mm, F.Cu at (167.5, -118.4)
- added TP8: GLOBAL_EN, TestPoint:TestPoint_Pad_D1.0mm, F.Cu at (185.9, -139.5)
- added TP9: FAN1, TestPoint:TestPoint_Pad_D1.0mm, F.Cu at (134.6, -85.5)
- added U1: TPD4EUSB30, Package_SON:USON-10_2.5x1.0mm_P0.5mm, F.Cu at (133.2, -81.2)
- added U10: SST25VF512A, Package_SO:SOIC-8_5.275x5.275mm_P1.27mm, F.Cu at (226.1, -116.3)
- added U11: TPD4EUSB30, Package_SON:USON-10_2.5x1.0mm_P0.5mm, F.Cu at (216.3, -107.1)
- added U12: TPD4EUSB30, Package_SON:USON-10_2.5x1.0mm_P0.5mm, F.Cu at (258.8, -135.6)
- added U13: AP62600, PintryParts-Footprints:V-QFN2030-12 (Type A), F.Cu at (118.3, -60.4)
- added U14: FSUSB30MUX, Package_SO:MSOP-10_3x3mm_P0.5mm, F.Cu at (235.7, -83.4)
- added U15: MIC2005-0.5LYM5, Package_TO_SOT_SMD:SOT-23-5, F.Cu at (222.3, -73.9)
- added U2: TPD4EUSB30, Package_SON:USON-10_2.5x1.0mm_P0.5mm, F.Cu at (194.5, -142.2)
- added U3: SN74LVC1G17, Package_TO_SOT_SMD:SOT-23-5, F.Cu at (129.8, -85.6)
- added U4: 74AHCT1G126, Package_TO_SOT_SMD:SOT-353_SC-70-5, F.Cu at (167.3, -114.2)
- added U5: TPD4EUSB30, Package_SON:USON-10_2.5x1.0mm_P0.5mm, F.Cu at (185.1, -135.2)
- added U6: TPD4EUSB30, Package_SON:USON-10_2.5x1.0mm_P0.5mm, F.Cu at (138.3, -85.8)
- added U7: ASM1061, PintryParts-Footprints:QFN-48-1EP_7x7mm_P0.5mm_EP4.025x4.025mm, F.Cu at (235.9, -115.1)
- added Y1: ECS-200-12-33-AGN-TR, Crystal:Crystal_SMD_3225-4Pin_3.2x2.5mm, F.Cu at (223.6, -110.6)
Other:
- board outline added: 100 x 100 mm
- copper layers 0 -> 4
