File: Pintry-X2/Pintry-X2.kicad_pcb (KiCad board)
At the start: 4 copper layers, 100 x 100 mm, 187 parts, among them J1 USB_B_Micro, J10 1735284-3, J11 54-00131, J12 Alternate Power Connector, J2 USB_A, J3 JD0-0001NL, J4 DM3D-SF, J5 UART, J6 Expansion, J7 Fan, J8 Fan, J9 1735284-3, Q1 BSS138PW, Q2 BSS138PW, Q5 SIA483DJ, Q6 BC857BW, Q7 SIA483DJ, SW1 SW_Push, U1 TPD4EUSB30, U10 SST25VF512A, U11 TPD4EUSB30, U12 TPD4EUSB30, U13 AP62600, U14 FSUSB30MUX, U15 MIC2005-0.5LYM5, U2 TPD4EUSB30, U3 SN74LVC1G17, U4 74AHCT1G126, U5 TPD4EUSB30, U6 TPD4EUSB30, U7 ASM1061, Y1 ECS-200-12-33-AGN-TR

Commit message: PCB Routing Complete - needs review
Parts:
- added Q3: BSS138PW, Package_TO_SOT_SMD:SOT-323_SC-70, F.Cu at (123.0, 191.4)
- added R16: 4K7, PintryParts-Footprints:R_0402_1005Metric, F.Cu at (122.3, 189.7)
- added R19: 1K, PintryParts-Footprints:R_0402_1005Metric, F.Cu at (77.1, 171.9)
- added R20: 1K, PintryParts-Footprints:R_0402_1005Metric, F.Cu at (77.1, 174.4)
- C1, C3, C41, C45, C46, C47, C48, C51, C52, C53, C54, D20, J7, R33, R34, U11, U12: moved to B.Cu
- Q5, Q7: footprint Package_TO_SOT_SMD:Vishay_PowerPAK_SC70-6L_Single -> PintryParts-Footprints:Vishay_PowerPAK_SC70-6L_Single
- TP1, TP10, TP11, TP14, TP16, TP17, TP18, TP2, TP3, TP4, TP5, TP6, TP7, TP8, TP9: footprint TestPoint:TestPoint_Pad_D1.0mm -> PintryParts-Footprints:TestPoint_Pad_D1.0mm
- TP15: footprint TestPoint:TestPoint_Pad_D1.0mm -> PintryParts-Footprints:TestPoint_Pad_D1.0mm; moved to B.Cu
- moved C9 347.7 mm to (81.4, 184.7), turned to 90 degrees
- moved SW1 346.4 mm to (143.6, 207.1), turned to 180 degrees
- moved U2 343.4 mm to (89.0, 184.6), turned to 90 degrees
- moved J3 338.1 mm to (87.1, 199.0)
- moved TP8 338.1 mm to (147.2, 196.3)
- moved C14 337.0 mm to (114.5, 207.7)
- moved D7 336.8 mm to (145.3, 201.9)
- moved U5 336.2 mm to (113.8, 193.3), turned to 90 degrees
- moved C49 335.5 mm to (106.9, 189.8), turned to 180 degrees
- moved R5 335.2 mm to (143.4, 201.9), turned to 180 degrees
- moved C12 335.1 mm to (145.4, 200.9)
- moved R15 330.0 mm to (143.4, 200.9), turned to 180 degrees
- moved C68 328.6 mm to (71.9, 170.2), turned to -90 degrees
- moved R14 326.2 mm to (147.0, 208.2)
- moved D17 325.5 mm to (148.8, 209.2), turned to 180 degrees
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Connections:
- net /CM4-USB-PCIe/~PCIe_RST renamed /CM4-USB-PCIe/~{PCIe_RST}
- J3 pad 4: /CM4-ETH-GPIO/ETH_1_P -> /CM4-ETH-GPIO/ETH_1_N
- J3 pad 5: /CM4-ETH-GPIO/ETH_1_N -> /CM4-ETH-GPIO/ETH_1_P
- J5 pad 1: /CM4-ETH-GPIO/RXD0 -> Net-(J5-Pad1)
- J5 pad 2: /CM4-ETH-GPIO/TXD0 -> Net-(J5-Pad2)
- J6 pad 1: /CM4-ETH-GPIO/GPIO10 -> +5V
- J6 pad 3: /CM4-ETH-GPIO/GPIO9 -> /CM4-ETH-GPIO/SCL1
- J6 pad 4: +5V -> /CM4-ETH-GPIO/SDA1
- J6 pad 5: /CM4-ETH-GPIO/GPIO11 -> /CM4-ETH-GPIO/GPIO10
- J6 pad 7: /CM4-ETH-GPIO/SCL1 -> /CM4-ETH-GPIO/GPIO9
- J6 pad 9: /CM4-ETH-GPIO/SDA1 -> /CM4-ETH-GPIO/GPIO11
- Module1 pad 93: /CM4-ETH-GPIO/~RPIBOOT -> /CM4-ETH-GPIO/~{RPIBOOT}
- U5 pad 1: /CM4-ETH-GPIO/SD_DAT2 -> unconnected-(U5-Pad1)
- U5 pad 10: /CM4-ETH-GPIO/SD_DAT2 -> unconnected-(U5-Pad1)
- U5 pad 2: /CM4-ETH-GPIO/SD_DAT3 -> /CM4-ETH-GPIO/SD_CMD
- U5 pad 4: /CM4-ETH-GPIO/SD_CLK -> /CM4-ETH-GPIO/SD_DAT3
- U5 pad 5: /CM4-ETH-GPIO/SD_CMD -> /CM4-ETH-GPIO/SD_DAT2
- U5 pad 6: /CM4-ETH-GPIO/SD_CMD -> /CM4-ETH-GPIO/SD_DAT2
- U5 pad 7: /CM4-ETH-GPIO/SD_CLK -> /CM4-ETH-GPIO/SD_DAT3
- U5 pad 9: /CM4-ETH-GPIO/SD_DAT3 -> /CM4-ETH-GPIO/SD_CMD
- U6 pad 1: /CM4-ETH-GPIO/SD_DAT0 -> /CM4-ETH-GPIO/SD_DAT1
- U6 pad 10: /CM4-ETH-GPIO/SD_DAT0 -> /CM4-ETH-GPIO/SD_DAT1
- U6 pad 2: /CM4-ETH-GPIO/SD_DAT1 -> /CM4-ETH-GPIO/SD_DAT0
- U6 pad 4: /CM4-ETH-GPIO/SDA1 -> /CM4-ETH-GPIO/SD_CLK
- U6 pad 5: /CM4-ETH-GPIO/SCL1 -> unconnected-(U6-Pad5)
- U6 pad 6: /CM4-ETH-GPIO/SCL1 -> unconnected-(U6-Pad5)
- U6 pad 7: /CM4-ETH-GPIO/SDA1 -> /CM4-ETH-GPIO/SD_CLK
- U6 pad 9: /CM4-ETH-GPIO/SD_DAT1 -> /CM4-ETH-GPIO/SD_DAT0
- U7 pad 49: (no net) -> GND
Routing:
- net +3V3: track 0.00 -> 359.1 mm, vias 0 -> 20
- net +12V: track 0.00 -> 214.9 mm, vias 0 -> 16
- net +5V: track 0.00 -> 138.1 mm, vias 0 -> 33
- net GND: track 0.00 -> 132.4 mm, vias 0 -> 309
- net /CM4-ETH-GPIO/PI_POWER_SW: track 0.00 -> 90.2 mm, vias 0 -> 4
- net /CM4-ETH-GPIO/ETH_0_P: track 0.00 -> 77.2 mm
- net /CM4-ETH-GPIO/ETH_0_N: track 0.00 -> 77.1 mm
- net /CM4-ETH-GPIO/RUN_PG: track 0.00 -> 73.1 mm, vias 0 -> 2
- net /CM4-ETH-GPIO/FAN1_PWM: track 0.00 -> 73.1 mm
- net /CM4-ETH-GPIO/PWR_LED: track 0.00 -> 71.8 mm, vias 0 -> 4
- net /CM4-USB-PCIe/USB_OTG: track 0.00 -> 68.9 mm, vias 0 -> 3
- net /CM4-ETH-GPIO/GLOBAL_EN: track 0.00 -> 68.4 mm, vias 0 -> 2
- net /CM4-ETH-GPIO/ETH_1_N: track 0.00 -> 67.9 mm
- net /CM4-ETH-GPIO/ETH_1_P: track 0.00 -> 67.8 mm
- net +1V2: track 0.00 -> 67.2 mm, vias 0 -> 8
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- added copper zone on F.Cu, net +12V
- added copper zone on F.Cu, net +1V2
- added copper zone on B.Cu, net +3V3
- added copper zone on F.Cu, net +5V
- added copper zone on In2.Cu, net +5V
- added copper zone on B.Cu, net GND
- added copper zone on F.Cu, net GND
- added copper zone on In1.Cu, net GND
- added copper zone on In2.Cu, net GND
- added copper zone on B.Cu, net Net-(C41-Pad1)
- added copper zone on F.Cu, net Net-(C41-Pad1)
- added copper zone on B.Cu, net Net-(C42-Pad1)
- added copper zone on F.Cu, net Net-(C42-Pad1)
- added copper zone on B.Cu, net Net-(C43-Pad1)
- added copper zone on F.Cu, net Net-(C43-Pad1)
- added copper zone on B.Cu, net Net-(C44-Pad1)
- added copper zone on F.Cu, net Net-(C44-Pad1)
- added copper zone on F.Cu, net Net-(C60-Pad2)
- added copper zone on F.Cu, net Net-(D24-Pad1)
- added copper zone on F.Cu, net Net-(FL1-Pad1)
- added copper zone on F.Cu, net Net-(FL1-Pad2)
- added copper zone on F.Cu, net Net-(FL1-Pad4)
Other:
- outline, holes or cut-outs redrawn
- board text added: "12V 6A MAX"
- board text added: "3V3"
- board text added: "5V"
- board text added: "GND"
- board text added: "P10"
- board text added: "P11"
- board text added: "P7"
- board text added: "P8"
- board text added: "P9"
- board text added: "Pintry X2"
- board text added: "RX"
- board text added: "Rev 1.0"
- board text added: "SCL"
- board text added: "SDA"
- board text added: "TX"
- board text added: "www.cezarchirila.com"
