File: Pintry-X2/CM4-ETH-GPIO.kicad_sch (KiCad schematic)
At the start: 60 parts, among them J3 JD0-0001NL, J4 DM3D-SF, J5 UART, J6 Expansion, J7 Fan, J8 Fan, Q1 BSS138PW, Q2 BSS138PW, SW1 SW_Push, U1 TPD4EUSB30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

Commit message: Moved ethernet connector so that it sticks out a bit
Parts:
- J7, J8: Part Number 0022232031 -> 47053-1000
Changed lines of the file:
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@@
       (effects (font (size 1.27 1.27)) hide)
     )
-    (property "Part Number" "0022232031" (id 5) (at 379.73 52.07 0)
+    (property "Part Number" "47053-1000" (id 5) (at 379.73 52.07 0)
       (effects (font (size 1.27 1.27)) hide)
     )
@@
       (effects (font (size 1.27 1.27)) hide)
     )
-    (property "Part Number" "0022232031" (id 5) (at 379.73 107.95 0)
+    (property "Part Number" "47053-1000" (id 5) (at 379.73 107.95 0)
       (effects (font (size 1.27 1.27)) hide)
     )
